File: custom ordered parts/breakout/breakout.kicad_pcb (KiCad board)
At the start: 2 copper layers, 55.5 x 50 mm, 28 parts

Commit message: Complete overhaul
Many changes are made, using more efficient/rigid components.
Parts:
- AUXF, AUXF1, AUXF3, HEF1, XTH0, XTH1, ZEND0, ZEND1: footprint Connector_JST:JST_XH_B2B-XH-A_1x02_P2.50mm_Vertical -> Tight Components:JST_XH_B2B-XH-A_1x02_P2.50mm_Vertical
- EM: renamed from EM1; footprint Connector_JST:JST_XH_B4B-XH-A_1x04_P2.50mm_Vertical -> Tight Components:JST_XH_B4B-XH-A_1x04_P2.50mm_Vertical
- FANPWM: renamed from FANPWM1; footprint Connector_JST:JST_XH_B2B-XH-A_1x02_P2.50mm_Vertical -> Tight Components:JST_XH_B2B-XH-A_1x02_P2.50mm_Vertical
- XEND: renamed from XEND1; footprint Connector_JST:JST_XH_B2B-XH-A_1x02_P2.50mm_Vertical -> Tight Components:JST_XH_B2B-XH-A_1x02_P2.50mm_Vertical
- XM0, XM1, YML0, YML1, YMR0, YMR1, ZM0, ZM1: footprint Connector_JST:JST_XH_B4B-XH-A_1x04_P2.50mm_Vertical -> Tight Components:JST_XH_B4B-XH-A_1x04_P2.50mm_Vertical
- YEND: renamed from YEND1; footprint Connector_JST:JST_XH_B2B-XH-A_1x02_P2.50mm_Vertical -> Tight Components:JST_XH_B2B-XH-A_1x02_P2.50mm_Vertical
- YTH: renamed from YTH1; footprint Connector_JST:JST_XH_B2B-XH-A_1x02_P2.50mm_Vertical -> Tight Components:JST_XH_B2B-XH-A_1x02_P2.50mm_Vertical
- moved YEND 0.21 mm to (194.7, 104.9)
- moved AUXF3 0.10 mm to (188.5, 80.1)
- moved YTH 0.10 mm to (195.7, 110.8)
- renumbered YR1 to YR
Routing:
- net Net-(JY1-Pin_4): track 21.7 -> 22.3 mm
